File: DIYTC2050PCB/DIYTC2050PCB.kicad_pcb (KiCad board)
At the start: 2 copper layers, 19.1 x 17 mm, 2 parts, among them J1 TC2050-IDC, J2 Conn_01x06_Pin

Commit message: Update PCB to a potential v2.0
Parts:
- added J3: Conn_01x04, Connector_PinSocket_2.54mm:PinSocket_1x04_P2.54mm_Vertical, F.Cu at (173.2, 80.0)
- J1: value TC2050-IDC -> TC2050; footprint THTTC2050Pogo:TagConnect2050 -> TC2050:TagConnect2050
- J2: value Conn_01x06_Pin -> Conn_01x04; footprint Connector_PinHeader_2.54mm:PinHeader_1x06_P2.54mm_Vertical -> Connector_PinSocket_2.54mm:PinSocket_1x04_P2.54mm_Vertical
- moved J2 32.0 mm to (173.2, 90.0)
- moved J1 29.3 mm to (177.1, 85.0)
Connections:
- net +3V3 renamed VCC
- J1 pad 2: SWDIO -> SWDIO/TMS
- J1 pad 4: SWDCLK -> SWCLK/TCK
- J1 pad 6: SWO -> SWO/TDO
- J1 pad 7: unconnected-(J1-Pad7) -> RTCLK
- J1 pad 8: unconnected-(J1-Pad8) -> TDI
- J2 pad 2: SWO -> SWDIO/TMS
- J2 pad 3: nRST -> SWCLK/TCK
- J2 pad 4: SWDIO -> nRST
Routing:
- net SWO: track 15.5 -> 0.00 mm
- net nRST: track 8.38 -> 16.8 mm
- net SWDCLK: track 6.58 -> 0.00 mm
- net SWDIO: track 6.58 -> 0.00 mm
- net TDI: track 0.00 -> 6.24 mm
- net RTCLK: track 0.00 -> 5.42 mm
- net GND: track 10.7 -> 5.45 mm, vias 0 -> 5
- net SWO/TDO: track 0.00 -> 4.89 mm
- net SWDIO/TMS: track 0.00 -> 4.36 mm
- net SWCLK/TCK: track 0.00 -> 4.36 mm
- net VCC: track 7.05 -> 4.89 mm
- added copper zone on B.Cu, net GND
- added copper zone on F.Cu, net GND
Other:
- board size 19.1 x 17 mm -> 15.2 x 20.5 mm
- board text added: "DIY TC2050 by"
- board text added: "JTAG"
- board text added: "P90Ez"
- board text added: "RTCLK"
- board text added: "SWCLK"
- board text added: "SWD/"
- board text added: "SWDIO"
- board text added: "TCK"
- board text added: "TDI"
- board text added: "TDO"
- board text added: "TMS"
- board text added: "Vref"
- board text removed: "P90s DIY TC2050"
- board text removed: "Rev1.1"
- board text removed: "SW CLK"
- board text removed: "SW DIO"
- board text removed: "VCC"
